File: inverter-igbt-driver.sch (KiCad schematic (older format))
At the start: 36 parts, among them J1 Conn_01x06, U1 NE555, U2 IXDF604SIA, U3 FOD8316, U6 Transformer_2P_2S

Commit message: Adds pull-down resistors for logic nets.
Parts:
- added R4, R5, R6, R7: 1k, Resistors_SMD:R_0402, symbol R
Connections:
- wire segments 100 -> 108
Other:
- note added: "Pull-Down Resistors"

Commit message: Add GND test point.
Parts:
- added TP5: TEST, inverter-igbt-driver:TP RCT (0805), symbol TEST
Changed lines of the file:
@@
 $EndComp
 $Comp
-L GND #PWR01
+L GND #PWR7
 U 1 1 5AC029A2
 P 3450 2800
-F 0 "#PWR01" H 3450 2550 50  0001 C CNN
+F 0 "#PWR7" H 3450 2550 50  0001 C CNN
 F 1 "GND" H 3450 2650 50  0000 C CNN
 F 2 "" H 3450 2800 50  0001 C CNN
@@
 $EndComp
 $Comp
-L +24V #PWR02
+L +24V #PWR6
 U 1 1 5AC029C6
 P 3450 1700
-F 0 "#PWR02" H 3450 1550 50  0001 C CNN
+F 0 "#PWR6" H 3450 1550 50  0001 C CNN
 F 1 "+24V" H 3450 1840 50  0000 C CNN
 F 2 "" H 3450 1700 50  0001 C CNN
@@
 $EndComp
 $Comp
-L +5V #PWR03
+L +5V #PWR1
 U 1 1 5AC0396A
 P 2100 1800
-F 0 "#PWR03" H 2100 1650 50  0001 C CNN
+F 0 "#PWR1" H 2100 1650 50  0001 C CNN
 F 1 "+5V" H 2100 1940 50  0000 C CNN
 F 2 "" H 2100 1800 50  0001 C CNN
@@
 $EndComp
 $Comp
-L GND #PWR04
+L GND #PWR2
 U 1 1 5AC03E97
 P 2100 2950
-F 0 "#PWR04" H 2100 2700 50  0001 C CNN
+F 0 "#PWR2" H 2100 2700 50  0001 C CNN
 F 1 "GND" H 2100 2800 50  0000 C CNN
 F 2 "" H 2100 2950 50  0001 C CNN
@@
 $EndComp
 $Comp
-L +5V #PWR05
+L +5V #PWR5
 U 1 1 5AC1BE5F
 P 2800 4250
-F 0 "#PWR05" H 2800 4100 50  0001 C CNN
+F 0 "#PWR5" H 2800 4100 50  0001 C CNN
 F 1 "+5V" H 2800 4390 50  0000 C CNN
 F 2 "" H 2800 4250 50  0001 C CNN
@@
 $EndComp
 $Comp
-L GND #PWR06
+L GND #PWR3
 U 1 1 5AC1C463
 P 2700 5050
-F 0 "#PWR06" H 2700 4800 50  0001 C CNN
+F 0 "#PWR3" H 2700 4800 50  0001 C CNN
 F 1 "GND" H 2700 4900 50  0000 C CNN
 F 2 "" H 2700 5050 50  0001 C CNN
@@
 Text Label 8250 4500 0    60   ~ 0
 VIN
-Text Notes 7600 3950 0    60   ~ 0
+Text Notes 7600 3900 0    60   ~ 0
 Incoming header for IO and Power Supply
 $Comp
@@
 $EndComp
 $Comp
-L GND #PWR07
+L GND #PWR4
 U 1 1 5ACCBED2
 P 2800 2750
-F 0 "#PWR07" H 2800 2500 50  0001 C CNN
+F 0 "#PWR4" H 2800 2500 50  0001 C CNN
 F 1 "GND" H 2800 2600 50  0000 C CNN
 F 2 "" H 2800 2750 50  0001 C CNN
@@
 Connection ~ 5150 4800
 Wire Wire Line
-	8450 4200 8250 4200
+	8150 4200 8450 4200
 Wire Wire Line
 	8450 4300 8250 4300
@@
 $EndComp
 $Comp
-L GND #PWR08
+L GND #PWR8
 U 1 1 5ACCE97E
 P 7950 5150
-F 0 "#PWR08" H 7950 4900 50  0001 C CNN
+F 0 "#PWR8" H 7950 4900 50  0001 C CNN
 F 1 "GND" H 7950 5000 50  0000 C CNN
 F 2 "" H 7950 5150 50  0001 C CNN
@@
 Text Notes 6800 4900 0    60   ~ 0
 Pull-Down Resistors
+$Comp
+L TEST TP5
+U 1 1 5ACD1B80
+P 8150 4200
+F 0 "TP5" H 8250 4350 50  0000 C BNN
+F 1 "TEST" H 8250 4450 50  0000 C CNN
+F 2 "inverter-igbt-driver:TP RCT (0805)" H 8150 4200 50  0001 C CNN
+F 3 "" H 8150 4200 50  0001 C CNN
+	1    8150 4200
+	1    0    0    -1
+$EndComp
 $EndSCHEMATC

Commit message: Switching pull-down to pull-up resistors for fault/reset.
Connections:
- wire segments 108 -> 109
Other:
- note added: "Pull-Up/Down Resistors"
- note removed: "Pull-Down Resistors"
- moved on the sheet: R4, R6, R7
Changed lines of the file:
@@
 $EndComp
 $Comp
-L GND #PWR7
+L GND #PWR01
 U 1 1 5AC029A2
 P 3450 2800
-F 0 "#PWR7" H 3450 2550 50  0001 C CNN
+F 0 "#PWR01" H 3450 2550 50  0001 C CNN
 F 1 "GND" H 3450 2650 50  0000 C CNN
 F 2 "" H 3450 2800 50  0001 C CNN
@@
 $EndComp
 $Comp
-L +24V #PWR6
+L +24V #PWR02
 U 1 1 5AC029C6
 P 3450 1700
-F 0 "#PWR6" H 3450 1550 50  0001 C CNN
+F 0 "#PWR02" H 3450 1550 50  0001 C CNN
 F 1 "+24V" H 3450 1840 50  0000 C CNN
 F 2 "" H 3450 1700 50  0001 C CNN
@@
 $EndComp
 $Comp
-L +5V #PWR1
+L +5V #PWR03
 U 1 1 5AC0396A
 P 2100 1800
-F 0 "#PWR1" H 2100 1650 50  0001 C CNN
+F 0 "#PWR03" H 2100 1650 50  0001 C CNN
 F 1 "+5V" H 2100 1940 50  0000 C CNN
 F 2 "" H 2100 1800 50  0001 C CNN
@@
 $EndComp
 $Comp
-L GND #PWR2
+L GND #PWR04
 U 1 1 5AC03E97
 P 2100 2950
-F 0 "#PWR2" H 2100 2700 50  0001 C CNN
+F 0 "#PWR04" H 2100 2700 50  0001 C CNN
 F 1 "GND" H 2100 2800 50  0000 C CNN
 F 2 "" H 2100 2950 50  0001 C CNN
@@
 $EndComp
 $Comp
-L +5V #PWR5
+L +5V #PWR05
 U 1 1 5AC1BE5F
 P 2800 4250
-F 0 "#PWR5" H 2800 4100 50  0001 C CNN
+F 0 "#PWR05" H 2800 4100 50  0001 C CNN
 F 1 "+5V" H 2800 4390 50  0000 C CNN
 F 2 "" H 2800 4250 50  0001 C CNN
@@
 $EndComp
 $Comp
-L GND #PWR3
+L GND #PWR06
 U 1 1 5AC1C463
 P 2700 5050
-F 0 "#PWR3" H 2700 4800 50  0001 C CNN
+F 0 "#PWR06" H 2700 4800 50  0001 C CNN
 F 1 "GND" H 2700 4900 50  0000 C CNN
 F 2 "" H 2700 5050 50  0001 C CNN
@@
 L R R4
 U 1 1 5ACCB4A7
-P 7800 4900
-F 0 "R4" V 7880 4900 50  0000 C CNN
-F 1 "1k" V 7800 4900 50  0000 C CNN
-F 2 "Resistors_SMD:R_0402" V 7730 4900 50  0001 C CNN
-F 3 "" H 7800 4900 50  0001 C CNN
-	1    7800 4900
+P 8050 4900
+F 0 "R4" V 8130 4900 50  0000 C CNN
+F 1 "1k" V 8050 4900 50  0000 C CNN
+F 2 "Resistors_SMD:R_0402" V 7980 4900 50  0001 C CNN
+F 3 "" H 8050 4900 50  0001 C CNN
+	1    8050 4900
 	1    0    0    -1
 $EndComp
@@
 $EndComp
 $Comp
-L GND #PWR4
+L GND #PWR07
 U 1 1 5ACCBED2
 P 2800 2750
-F 0 "#PWR4" H 2800 2500 50  0001 C CNN
+F 0 "#PWR07" H 2800 2500 50  0001 C CNN
 F 1 "GND" H 2800 2600 50  0000 C CNN
 F 2 "" H 2800 2750 50  0001 C CNN
@@
 Wire Wire Line
 	8450 4400 8250 4400
-Wire Wire Line
-	7800 4500 8450 4500
-Wire Wire Line
-	7950 4600 8450 4600
-Wire Wire Line
-	8100 4700 8450 4700
 Connection ~ 2800 2350
 Wire Wire Line
@@
 L R R6
 U 1 1 5ACCE827
-P 7950 4900
-F 0 "R6" V 8030 4900 50  0000 C CNN
-F 1 "1k" V 7950 4900 50  0000 C CNN
-F 2 "Resistors_SMD:R_0402" V 7880 4900 50  0001 C CNN
-F 3 "" H 7950 4900 50  0001 C CNN
-	1    7950 4900
+P 7750 4350
+F 0 "R6" V 7830 4350 50  0000 C CNN
+F 1 "1k" V 7750 4350 50  0000 C CNN
+F 2 "Resistors_SMD:R_0402" V 7680 4350 50  0001 C CNN
+F 3 "" H 7750 4350 50  0001 C CNN
+	1    7750 4350
 	1    0    0    -1
 $EndComp
@@
 L R R7
 U 1 1 5ACCE8BE
-P 8100 4900
-F 0 "R7" V 8180 4900 50  0000 C CNN
-F 1 "1k" V 8100 4900 50  0000 C CNN
-F 2 "Resistors_SMD:R_0402" V 8030 4900 50  0001 C CNN
-F 3 "" H 8100 4900 50  0001 C CNN
-	1    8100 4900
-	1    0    0    -1
-$EndComp
-$Comp
-L GND #PWR8
+P 7950 4350
+F 0 "R7" V 8030 4350 50  0000 C CNN
+F 1 "1k" V 7950 4350 50  0000 C CNN
+F 2 "Resistors_SMD:R_0402" V 7880 4350 50  0001 C CNN
+F 3 "" H 7950 4350 50  0001 C CNN
+	1    7950 4350
+	1    0    0    -1
+$EndComp
+$Comp
+L GND #PWR08
 U 1 1 5ACCE97E
-P 7950 5150
-F 0 "#PWR8" H 7950 4900 50  0001 C CNN
-F 1 "GND" H 7950 5000 50  0000 C CNN
-F 2 "" H 7950 5150 50  0001 C CNN
-F 3 "" H 7950 5150 50  0001 C CNN
-	1    7950 5150
-	1    0    0    -1
-$EndComp
-Wire Wire Line
-	7800 5050 7800 5100
-Wire Wire Line
-	7800 5100 8100 5100
-Wire Wire Line
-	8100 5100 8100 5050
-Wire Wire Line
-	7950 5050 7950 5150
-Connection ~ 7950 5100
-Wire Wire Line
-	8100 4750 8100 4700
-Wire Wire Line
-	7950 4750 7950 4600
-Wire Wire Line
-	7800 4750 7800 4500
-Text Notes 6800 4900 0    60   ~ 0
-Pull-Down Resistors
+P 8050 5100
+F 0 "#PWR08" H 8050 4850 50  0001 C CNN
+F 1 "GND" H 8050 4950 50  0000 C CNN
+F 2 "" H 8050 5100 50  0001 C CNN
+F 3 "" H 8050 5100 50  0001 C CNN
+	1    8050 5100
+	1    0    0    -1
+$EndComp
+Text Notes 6600 4650 0    60   ~ 0
+Pull-Up/Down Resistors
 $Comp
 L TEST TP5
@@
 	1    0    0    -1
 $EndComp
+Wire Wire Line
+	7950 4600 8450 4600
+Wire Wire Line
+	7950 4600 7950 4500
+Wire Wire Line
+	7750 4700 8450 4700
+Wire Wire Line
+	7750 4700 7750 4500
+Wire Wire Line
+	8050 4500 8450 4500
+Wire Wire Line
+	8050 4500 8050 4750
+Wire Wire Line
+	8050 5050 8050 5100
+$Comp
+L +5V #PWR?
+U 1 1 5ACD9AA7
+P 7850 4100
+F 0 "#PWR?" H 7850 3950 50  0001 C CNN
+F 1 "+5V" H 7850 4240 50  0000 C CNN
+F 2 "" H 7850 4100 50  0001 C CNN
+F 3 "" H 7850 4100 50  0001 C CNN
+	1    7850 4100
+	1    0    0    -1
+$EndComp
+Wire Wire Line
+	7750 4200 7750 4150
+Wire Wire Line
+	7750 4150 7950 4150
+Wire Wire Line
+	7950 4150 7950 4200
+Wire Wire Line
+	7850 4100 7850 4150
+Connection ~ 7850 4150
 $EndSCHEMATC

Commit message: Refactor into schematic.
Parts:
- removed C1: 0.01u, Capacitors_SMD:C_0603_HandSoldering, symbol C
- removed C10, C11, C12, C2, C3, C4, C5, C6, C7, C8, C9: 10u, Capacitors_SMD:C_1206_HandSoldering, symbol C
- removed C13: 100p, Capacitors_SMD:C_1206_HandSoldering, symbol C
- removed COLL1, EMIT1, GATE1: Conn_01x01, inverter-igbt-driver:CONN_110_TAB, symbol Conn_01x01
- removed D1, D2, D3: D_Schottky, Diodes_SMD:D_SOD-123F, symbol D_Schottky
- removed D4: D, inverter-igbt-driver:DO-214AC, symbol D
- removed R1: 1.5k, Resistors_SMD:R_0603_HandSoldering, symbol R
- removed R2: 100, Resistors_SMD:R_1206_HandSoldering, symbol R
- removed R3: 8, Resistors_THT:R_Axial_DIN0207_L6.3mm_D2.5mm_P7.62mm_Horizontal, symbol R
- removed R5: 1k, Resistors_SMD:R_0402, symbol R
- removed TP1, TP2, TP3, TP4, TP6, TP7, TP8, TP9: TEST, inverter-igbt-driver:TP RCT (0805), symbol TEST
- removed U1: NE555, Housings_SOIC:SOIC-8_3.9x4.9mm_Pitch1.27mm, symbol NE555
- removed U2: IXDF604SIA, Housings_SOIC:SOIC-8_3.9x4.9mm_Pitch1.27mm, symbol IXDF604SIA
- removed U3: FOD8316, Housings_SOIC:SOIC-16W_7.5x10.3mm_Pitch1.27mm, symbol FOD8316
- removed U6: Transformer_2P_2S, inverter-igbt-driver:FS48-050-C2, symbol Transformer_2P_2S
Connections:
- net labels added: COLL, EMIT, GATE
- net labels removed: VDD_IGBT, VE_IGBT, VSS_IGBT
- wire segments 109 -> 20
Other:
- note removed: "+15/-8V Power Supply for IGBT Driver\n"
- note removed: "24V Square Wave @ 48kHz"
- note removed: "Generates 48kHz Square Wave\nf = 1.44 / (2 * 1.5k * 0.01u) = 48k"
- note removed: "Greinacher voltage doubler\nDoubles and rectifies secondary voltage"
- note removed: "IGBT Driver With Desaturation Fault Handling"
- note removed: "Rectifies voltage on negative swing"
- note removed: "XFMR Provides HV Isolation\nTurns ratio reduces 24V to 8V VDD\n\nPrimary Windings are 115V (2 in parallel)\nSecondary Windings are 24V (2 in series)\nEffective Turns Ratio == 115:48 == 2.4"
- moved on the sheet: R4, R6, R7, TP5

Commit message: Including both igbt drivers on one board.
WIP
Parts:
- added J2: Conn_01x06, Pin_Headers:Pin_Header_Straight_1x06_Pitch1.00mm, symbol Conn_01x06
- added R10, R8, R9: 1k, Resistors_SMD:R_0402, symbol R
- added TP10: TEST, inverter-igbt-driver:TP RCT (0805), symbol TEST
- added U?: IGBT_HALF_BRIDGE, symbol IGBT_HALF_BRIDGE
Connections:
- net labels added: COLL_L, EMIT_L, FAULT_L, GATE_L, RESET_L, VIN_L
- wire segments 20 -> 48
Other:
- moved on the sheet: R4, R6, R7, TP5

Commit message: Add _H suffix to hot leg.
Parts:
- U9: renamed from U?; footprint (none) -> inverter-igbt-driver:MG06600WB-BN4MM
Connections:
- net labels added: COLL_H, EMIT_H, FAULT_H, GATE_H, RESET_H, VIN_H
- net labels removed: COLL, EMIT, FAULT, GATE, RESET, VIN
Changed lines of the file:
@@
 +24V
 Text Label 2850 2450 0    60   ~ 0
-FAULT
+FAULT_H
 Text Label 2850 2550 0    60   ~ 0
-RESET
+RESET_H
 Text Label 2850 2350 0    60   ~ 0
-VIN
+VIN_H
 Text Notes 2200 1750 0    60   ~ 0
 Incoming header for IO and Power Supply
@@
 $EndSheet
 Text Label 4900 2350 2    60   ~ 0
-VIN
+VIN_H
 Text Label 4900 2500 2    60   ~ 0
-RESET
+RESET_H
 Text Label 4900 2650 2    60   ~ 0
-FAULT
+FAULT_H
 Wire Wire Line
 	4900 2350 5100 2350
@@
 	4900 2650 5100 2650
 Text Label 6300 2350 0    60   ~ 0
-COLL
+COLL_H
 Text Label 6300 2500 0    60   ~ 0
-GATE
+GATE_H
 Text Label 6300 2650 0    60   ~ 0
-EMIT
+EMIT_H
 Wire Wire Line
 	6100 2350 6950 2350
@@
 Connection ~ 2450 3550
 $Comp
-L IGBT_HALF_BRIDGE U?
+L IGBT_HALF_BRIDGE U9
 U 1 1 5ADAB658
 P 7500 3000
-F 0 "U?" H 8350 4200 60  0000 C CNN
+F 0 "U9" H 8350 4200 60  0000 C CNN
 F 1 "IGBT_HALF_BRIDGE" H 7700 4200 60  0000 C CNN
-F 2 "" H 7700 2950 60  0001 C CNN
+F 2 "inverter-igbt-driver:MG06600WB-BN4MM" H 7700 2950 60  0001 C CNN
 F 3 "" H 7700 2950 60  0001 C CNN
 	1    7500 3000

Commit message: Move square wave generator to single module.
Connections:
- wire segments 48 -> 54
Other:
- moved on the sheet: U9
Changed lines of the file:
@@
 $Descr A4 11693 8268
 encoding utf-8
-Sheet 1 3
+Sheet 1 4
 Title "3 Phase Inverter IGBT Driver For Single Half Bridge"
 Date "2018-04-02"
@@
 Connection ~ 2450 2000
 $Sheet
-S 5100 2150 1000 800
+S 7050 1950 1000 800
 U 5AD96A61
 F0 "positive" 60
 F1 "positive.sch" 60
-F2 "COLL" I R 6100 2350 60
-F3 "GATE" I R 6100 2500 60
-F4 "EMIT" I R 6100 2650 60
-F5 "VIN" I L 5100 2350 60
-F6 "RESET" I L 5100 2500 60
-F7 "FAULT" I L 5100 2650 60
+F2 "COLL" I R 8050 2150 60
+F3 "GATE" I R 8050 2300 60
+F4 "EMIT" I R 8050 2450 60
+F5 "VIN" I L 7050 2050 60
+F6 "RESET" I L 7050 2150 60
+F7 "FAULT" I L 7050 2250 60
+F8 "SQUARE_H" I L 7050 2450 60
+F9 "SQUARE_L" I L 7050 2550 60
 $EndSheet
-Text Label 4900 2350 2    60   ~ 0
+Text Label 6850 2050 2    60   ~ 0
 VIN_H
-Text Label 4900 2500 2    60   ~ 0
+Text Label 6850 2150 2    60   ~ 0
 RESET_H
-Text Label 4900 2650 2    60   ~ 0
+Text Label 6850 2250 2    60   ~ 0
 FAULT_H
 Wire Wire Line
-	4900 2350 5100 2350
-Wire Wire Line
-	4900 2500 5100 2500
-Wire Wire Line
-	4900 2650 5100 2650
-Text Label 6300 2350 0    60   ~ 0
+	6850 2050 7050 2050
+Wire Wire Line
+	6850 2150 7050 2150
+Wire Wire Line
+	6850 2250 7050 2250
+Text Label 8250 2150 0    60   ~ 0
 COLL_H
-Text Label 6300 2500 0    60   ~ 0
+Text Label 8250 2300 0    60   ~ 0
 GATE_H
-Text Label 6300 2650 0    60   ~ 0
+Text Label 8250 2450 0    60   ~ 0
 EMIT_H
 Wire Wire Line
-	6100 2350 6950 2350
-Wire Wire Line
-	6100 2500 6750 2500
-Wire Wire Line
-	6100 2650 6650 2650
+	8050 2150 8900 2150
+Wire Wire Line
+	8050 2300 8700 2300
+Wire Wire Line
+	8050 2450 8600 2450
 $Sheet
-S 5100 3150 1000 750
+S 7050 2950 1000 750
 U 5ADA6656
 F0 "negative" 60
 F1 "positive.sch" 60
-F2 "COLL" I R 6100 3350 60
-F3 "GATE" I R 6100 3500 60
-F4 "EMIT" I R 6100 3650 60
-F5 "VIN" I L 5100 3350 60
-F6 "RESET" I L 5100 3500 60
-F7 "FAULT" I L 5100 3650 60
+F2 "COLL" I R 8050 3150 60
+F3 "GATE" I R 8050 3300 60
+F4 "EMIT" I R 8050 3450 60
+F5 "VIN" I L 7050 3050 60
+F6 "RESET" I L 7050 3150 60
+F7 "FAULT" I L 7050 3250 60
+F8 "SQUARE_H" I L 7050 3450 60
+F9 "SQUARE_L" I L 7050 3550 60
 $EndSheet
-Text Label 4900 3350 2    60   ~ 0
+Text Label 6850 3050 2    60   ~ 0
 VIN_L
-Text Label 4900 3500 2    60   ~ 0
+Text Label 6850 3150 2    60   ~ 0
 RESET_L
-Text Label 4900 3650 2    60   ~ 0
+Text Label 6850 3250 2    60   ~ 0
 FAULT_L
-Text Label 6300 3350 0    60   ~ 0
+Text Label 8250 3150 0    60   ~ 0
 COLL_L
-Text Label 6300 3500 0    60   ~ 0
+Text Label 8250 3300 0    60   ~ 0
 GATE_L
-Text Label 6300 3650 0    60   ~ 0
+Text Label 8250 3450 0    60   ~ 0
 EMIT_L
 Wire Wire Line
-	6100 3350 6650 3350
-Wire Wire Line
-	6100 3500 6750 3500
-Wire Wire Line
-	6100 3650 6950 3650
-Wire Wire Line
-	5100 3350 4900 3350
-Wire Wire Line
-	4900 3500 5100 3500
-Wire Wire Line
-	5100 3650 4900 3650
+	8600 3150 8050 3150
+Wire Wire Line
+	8050 3300 8700 3300
+Wire Wire Line
+	8050 3450 8900 3450
+Wire Wire Line
+	7050 3050 6850 3050
+Wire Wire Line
+	6850 3150 7050 3150
+Wire Wire Line
+	7050 3250 6850 3250
 $Comp
 L Conn_01x06 J2
@@
 L IGBT_HALF_BRIDGE U9
 U 1 1 5ADAB658
-P 7500 3000
-F 0 "U9" H 8350 4200 60  0000 C CNN
-F 1 "IGBT_HALF_BRIDGE" H 7700 4200 60  0000 C CNN
-F 2 "inverter-igbt-driver:MG06600WB-BN4MM" H 7700 2950 60  0001 C CNN
-F 3 "" H 7700 2950 60  0001 C CNN
-	1    7500 3000
-	1    0    0    -1
-$EndComp
-Wire Wire Line
-	6650 3350 6650 2650
-Wire Wire Line
-	6950 3000 6650 3000
-Connection ~ 6650 3000
-Wire Wire Line
-	6950 2850 6750 2850
-Wire Wire Line
-	6750 2850 6750 2500
-Wire Wire Line
-	6950 3350 6750 3350
-Wire Wire Line
-	6750 3350 6750 3500
-Wire Wire Line
-	6950 2350 6950 2450
-Wire Wire Line
-	6950 3650 6950 3550
+P 9450 2800
+F 0 "U9" H 10300 4000 60  0000 C CNN
+F 1 "IGBT_HALF_BRIDGE" H 9650 4000 60  0000 C CNN
+F 2 "inverter-igbt-driver:MG06600WB-BN4MM" H 9650 2750 60  0001 C CNN
+F 3 "" H 9650 2750 60  0001 C CNN
+	1    9450 2800
+	1    0    0    -1
+$EndComp
+Wire Wire Line
+	8600 2450 8600 3150
+Wire Wire Line
+	8900 2800 8600 2800
+Connection ~ 8600 2800
+Wire Wire Line
+	8900 2650 8700 2650
+Wire Wire Line
+	8700 2650 8700 2300
+Wire Wire Line
+	8900 3150 8700 3150
+Wire Wire Line
+	8700 3150 8700 3300
+Wire Wire Line
+	8900 2150 8900 2250
+Wire Wire Line
+	8900 3450 8900 3350
+$Sheet
+S 4900 2250 650  550
+U 5ADB7652
+F0 "square_wave_generator" 60
+F1 "square_wave_generator.sch" 60
+F2 "SQUARE_H" I R 5550 2450 60
+F3 "SQUARE_L" I R 5550 2550 60
+$EndSheet
+Wire Wire Line
+	5550 2450 7050 2450
+Wire Wire Line
+	7000 2550 5550 2550
+Wire Wire Line
+	7050 3450 6450 3450
+Wire Wire Line
+	6450 3450 6450 2450
+Connection ~ 6450 2450
+Wire Wire Line
+	7050 3550 6400 3550
+Wire Wire Line
+	6400 3550 6400 2550
+Connection ~ 6400 2550
 $EndSCHEMATC

Commit message: Fixing layout
Parts:
- removed TP10: TEST, inverter-igbt-driver:TP RCT (0805), symbol TEST
Changed lines of the file:
@@
 $EndComp
-Wire Wire Line
-	2750 3600 3050 3600
 Wire Wire Line
 	3050 3700 2850 3700
@@
 Text Notes 1200 4050 0    60   ~ 0
 Pull-Up/Down Resistors
-$Comp
-L TEST TP10
-U 1 1 5ADA812D
-P 2750 3600
-F 0 "TP10" H 2850 3750 50  0000 C BNN
-F 1 "TEST" H 2850 3850 50  0000 C CNN
-F 2 "inverter-igbt-driver:TP RCT (0805)" H 2750 3600 50  0001 C CNN
-F 3 "" H 2750 3600 50  0001 C CNN
-	1    2750 3600
-	1    0    0    -1
-$EndComp
 Wire Wire Line
 	2550 4000 3050 4000
@@
 	6400 3550 6400 2550
 Connection ~ 6400 2550
+Wire Wire Line
+	3050 3600 2850 3600
 $EndSCHEMATC
