File: inverter-igbt-driver.kicad_pcb (KiCad board)
At the start: 2 copper layers, 84.5 x 64 mm, 70 parts, among them J1 CONTROL, U1 NE555, U2 IXDF604SIA, U3 FOD8316, U4 74LVC1G80GV, U5 FOD8316, U6 Transformer_2P_2S, U8 Transformer_2P_2S, U9 IGBT_HALF_BRIDGE

Commit message: Update values.
Parts:
- C1: value 0.01u -> 0.001n
- R11: value 1.5k -> 5.6k
Connections:
- U4 pad 4: Net-(R5-Pad1) -> (no net)
